Commit message: MoveIt Packages and URDF Modifications

File: mycobot_description/urdf/mycobot_280_m5/mycobot_280m5_with_gripper_parallel.urdf (robot description, URDF)
Before this commit: robot firefighter, 15 links, 14 joints
Links:
- link g_base: mass 0.1 -> None
- link gripper_base: mass 0.1 -> None; geometry collision mesh filename=package://mycobot_description/urdf/mycobot_280_m5/gripper_b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; visual mesh filename=package://mycobot_description/urdf/mycobot_280_m5/gripper_b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
- link gripper_left1: mass 0.1 -> None; geometry collision mesh filename=package://mycobot_description/urdf/mycobot_280_m5/gripper_l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; visual mesh filename=package://mycobot_description/urdf/mycobot_280_m5/gripper_l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
- link gripper_left2: mass 0.1 -> None; geometry collision mesh filename=package://mycobot_description/urdf/mycobot_280_m5/gripper_l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; visual mesh filename=package://mycobot_description/urdf/mycobot_280_m5/gripper_l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
- link gripper_left3: mass 0.1 -> None; geometry collision mesh filename=package://mycobot_description/urdf/mycobot_280_m5/gripper_l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; visual mesh filename=package://mycobot_description/urdf/mycobot_280_m5/gripper_l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
- link gripper_right1: mass 0.1 -> None; geometry collision mesh filename=package://mycobot_description/urdf/mycobot_280_m5/gripper_r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; visual mesh filename=package://mycobot_description/urdf/mycobot_280_m5/gripper_r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
- link gripper_right2: mass 0.1 -> None; geometry collision mesh filename=package://mycobot_description/urdf/mycobot_280_m5/gripper_r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; visual mesh filename=package://mycobot_description/urdf/mycobot_280_m5/gripper_r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
- link gripper_right3: mass 0.1 -> None; geometry collision mesh filename=package://mycobot_description/urdf/mycobot_280_m5/gripper_r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; visual mesh filename=package://mycobot_description/urdf/mycobot_280_m5/gripper_r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
- link joint1: mass 0.1 -> None
- link joint2: mass 0.1 -> None
- link joint3: mass 0.1 -> None
- link joint4: mass 0.1 -> None
- link joint5: mass 0.1 -> None
- link joint6: mass 0.1 -> None
- link joint6_flange: mass 0.1 -> None
Joints:
- joint gripper_controller: limit lower=-0.78 upper=0.15 effort=1000.0 velocity=0 -> lower=-0.7 upper=0.15 effort=1000.0 velocity=0
